File: hw/coop_door.kicad_sch (KiCad schematic)
At the start: 53 parts, among them J1 Screw_Terminal_01x02, J2 Screw_Terminal_01x02, J3 Screw_Terminal_01x02, Q1 IRLTS6342, Q2 IRF4905, Q3 IRLTS6342, Q4 BSD235NH, Q5 BSL207SPH, SW1 SW_Push, SW2 SW_DPDT_x2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

Commit message: Update schematics&PCB
- Add button to start the battery protection IC
- Add motor resitor to AISEN pin to limit the current to ~300mA
Parts:
- removed C5: 10n, Capacitor_THT:C_Rect_L7.0mm_W4.5mm_P5.00mm, symbol Device:C
- removed C6: 2.2u, Capacitor_THT:CP_Radial_D4.0mm_P2.00mm, symbol Device:C_Polarized
- removed C8: 10u, Capacitor_THT:C_Rect_L7.0mm_W4.5mm_P5.00mm, symbol Device:C
- removed J1: Screw_Terminal_01x02, TerminalBlock:TerminalBlock_Altech_AK300-2_P5.00mm, symbol Connector:Screw_Terminal_01x02
- removed R7: 1k, Resistor_THT:R_Axial_DIN0207_L6.3mm_D2.5mm_P7.62mm_Horizontal, symbol Device:R
- removed R9: 10k, Resistor_THT:R_Axial_DIN0207_L6.3mm_D2.5mm_P7.62mm_Horizontal, symbol Device:R
- removed U3: DRV8833PW, Package_SO:TSSOP-16_4.4x5mm_P0.65mm, symbol Driver_Motor:DRV8833PW
- added C14: 2.2u, Capacitor_THT:CP_Radial_D4.0mm_P2.00mm, symbol Device:C_Polarized
- added C15: 10u, Capacitor_THT:C_Rect_L7.0mm_W4.5mm_P5.00mm, symbol Device:C
- added C6: 10n, Capacitor_THT:C_Rect_L7.0mm_W4.5mm_P5.00mm, symbol Device:C
- added J4: Screw_Terminal_01x02, TerminalBlock:TerminalBlock_Altech_AK300-2_P5.00mm, symbol Connector:Screw_Terminal_01x02
- added R20: 0R68, Resistor_THT:R_Axial_DIN0207_L6.3mm_D2.5mm_P7.62mm_Horizontal, symbol Device:R
- added R21: 1k, Resistor_THT:R_Axial_DIN0207_L6.3mm_D2.5mm_P7.62mm_Horizontal, symbol Device:R
- added R22: 10k, Resistor_THT:R_Axial_DIN0207_L6.3mm_D2.5mm_P7.62mm_Horizontal, symbol Device:R
- added SW3: SW_Push, Button_Switch_THT:SW_PUSH_6mm, symbol Switch:SW_Push
- added U6: DRV8833PW, Package_SO:TSSOP-16_4.4x5mm_P0.65mm, symbol coop_door_library:DRV8833PW
- U4: footprint coop_door_footprints:RPi_Pico_SMD_TH -> RPi_Pico:RPi_Pico_SMD_TH
- U5: footprint Package_TO_SOT_SMD:SOT-23-6_Handsoldering -> Package_TO_SOT_SMD:SOT-23-6
Connections:
- net +BATT: now also C15.2, C6.1, U6.12 (VM)
- net GND: now also C14.2, C15.1, R20.1, R22.2, U6.13 (GND), U6.6 (BISEN)
- net motor_drv_AIN1: now also U6.16 (AIN1)
- net motor_drv_AIN2: now also U6.15 (AIN2)
- net motor_drv_AOUT1: now also J4.1 (Pin_1), U6.2 (AOUT1)
- net motor_drv_AOUT2: now also J4.2 (Pin_2), U6.4 (AOUT2)
- net motor_drv_nFAULT: now also U6.8 (~{FAULT})
- net motor_drv_nSLEEP: now also R21.2
- net at BT3.2 (-), C10.2, C13.2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: now also SW3.1
- net at Q4.2 (G), U5.1 (DO): now also SW3.2
- new net: R21.1, R22.1, U6.1 (~{SLEEP})
- new net: C6.2, U6.11 (VCP)
- new net: C14.1, U6.14 (VINT)
- new net motor_drv_AISEN: R20.2, U6.3 (AISEN)
Other:
- moved on the sheet: BT2, BT3, C10, C13, C9, Q4A, Q4B, R15, R16, R17, U5
